File: PCB/TeensyPicoCap4/TeensyPicoCap4.kicad_sch (KiCad schematic)
At the start: 42 parts, among them J1 Conn_01x02, J10 Conn_01x01_Male, J11 Conn_01x01_Male, J12 Conn_01x01_Male, J13 Conn_01x01_Male, J14 Conn_01x24, J15 Conn_01x24, J16 Barrel_Jack_Switch_Pin3Ring, J17 Conn_01x08, J18 Conn_01x08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

Commit message: submitted V1 w/ more silk and digikey parts
Parts:
- C4: Digikey (none) -> 399-C320C104K5R5TA7305CT-ND
- F1: Digikey (none) -> F2112CT-ND
- J1, J2, J3: Digikey (none) -> 2057-EBWA-02-B-ND
- R2: Digikey TT-PT-1000A-2050-11-AUNI-ND -> 223-1807-ND
Changed lines of the file:
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@@
+      (effects (font (size 1.27 1.27)) hide)
+    )
+    (property "Digikey" "F2112CT-ND" (id 4) (at 237.49 31.75 0)
       (effects (font (size 1.27 1.27)) hide)
     )
@@
       (effects (font (size 1.27 1.27)) hide)
     )
-    (property "Datasheet" "~" (id 3) (at 80.01 95.25 0)
-      (effects (font (size 1.27 1.27)) hide)
-    )
-    (property "Digikey" "TT-PT-1000A-2050-11-AUNI-ND" (id 4) (at 80.01 95.25 0)
+    (property "Datasheet" "https://www.digikey.com/en/products/detail/te-connectivity-measurement-specialties/NB-PTCO-157/5272171" (id 3) (at 80.01 95.25 0)
+      (effects (font (size 1.27 1.27)) hide)
+    )
+    (property "Digikey" "223-1807-ND" (id 4) (at 80.01 95.25 0)
       (effects (font (size 1.27 1.27)) hide)
     )
@@
       (effects (font (size 1.27 1.27)) hide)
     )
-    (property "Datasheet" "~" (id 3) (at 43.18 77.47 0)
+    (property "Datasheet" "https://www.digikey.com/en/products/detail/adam-tech/EBWA-02-B/9830632" (id 3) (at 43.18 77.47 0)
+      (effects (font (size 1.27 1.27)) hide)
+    )
+    (property "Digikey" "2057-EBWA-02-B-ND" (id 4) (at 43.18 77.47 0)
       (effects (font (size 1.27 1.27)) hide)
     )
@@
       (effects (font (size 1.27 1.27)) hide)
     )
-    (property "Datasheet" "~" (id 3) (at 43.18 67.31 0)
+    (property "Datasheet" "https://www.digikey.com/en/products/detail/adam-tech/EBWA-02-B/9830632" (id 3) (at 43.18 67.31 0)
+      (effects (font (size 1.27 1.27)) hide)
+    )
+    (property "Digikey" "2057-EBWA-02-B-ND" (id 4) (at 43.18 67.31 0)
       (effects (font (size 1.27 1.27)) hide)
     )
@@
     )
     (property "Datasheet" "~" (id 3) (at 81.28 162.56 0)
+      (effects (font (size 1.27 1.27)) hide)
+    )
+    (property "Digikey" "399-C320C104K5R5TA7305CT-ND" (id 4) (at 81.28 162.56 0)
       (effects (font (size 1.27 1.27)) hide)
     )
@@
       (effects (font (size 1.27 1.27)) hide)
     )
-    (property "Datasheet" "~" (id 3) (at 43.18 87.63 0)
-      (effects (font (size 1.27 1.27)) hide)
-    )
+    (property "Datasheet" "https://www.digikey.com/en/products/detail/adam-tech/EBWA-02-B/9830632" (id 3) (at 43.18 87.63 0)
+      (effects (font (size 1.27 1.27)) hide)
+    )
+    (property "Digikey" "2057-EBWA-02-B-ND" (id 4) (at 43.18 87.63 0)
+      (effects (font (size 1.27 1.27)) hide)
+    )
